Commit message: fixed angle grip. added random positioning

File: temp_01.urdf (robot description, URDF)
Before this commit: robot test_joint, 8 links, 7 joints
Links:
- link stand_leg: geometry collision box size=0.1 0.1 1.2
Joints:
- joint stand_arm_joint: axis 0.5 1.25 0 -> (none); type continuous -> fixed
- joint stand_foot_joint: axis 0 1 0 -> (none); type continuous -> fixed

Commit message: prismatic joints

File: temp_01.urdf (robot description, URDF)
Before this commit: robot test_joint, 8 links, 7 joints
Links:
- link stand_arm: geometry collision box size=0.1 0.5 0.1
Joints:
- joint stand_arm_joint: origin xyz=0 1.0 0 rpy=0 0 0 -> xyz=0 0.6 0 rpy=0 0 0
- joint stand_leg_joint: axis 1 0 0 -> 0 0 1; limit (none) -> lower=0 upper=-1.2; type continuous -> prismatic

Commit message: created loop to test robustness

File: temp_01.urdf (robot description, URDF)
Before this commit: robot test_joint, 8 links, 7 joints
Links:
- added link left_contact_1, mass 0.2; collision box size=0.05 0.1 0.2
- added link left_contact_2, mass 0.2; collision box size=0.05 0.1 0.2
- added link left_contact_3, mass 0.2; collision box size=0.05 0.1 0.2
- added link left_contact_4, mass 0.2; collision box size=0.05 0.1 0.2
- added link right_contact_1, mass 0.2; collision box size=0.05 0.1 0.2
- added link right_contact_2, mass 0.2; collision box size=0.05 0.1 0.2
- added link right_contact_3, mass 0.2; collision box size=0.05 0.1 0.2
- added link right_contact_4, mass 0.2; collision box size=0.05 0.1 0.2
Joints:
- added joint left_joint_1: type prismatic, parent left_forearm, child left_contact_1, origin xyz=-0.3 0 -0.1 rpy=0 0 0, axis 0 0 1, limit lower=0 upper=1
- added joint left_joint_2: type prismatic, parent left_forearm, child left_contact_2, origin xyz=-0.25 0 -0.1 rpy=0 0 0, axis 0 0 1, limit lower=0 upper=1
- added joint left_joint_3: type prismatic, parent left_forearm, child left_contact_3, origin xyz=-0.19999999999999998 0 -0.1 rpy=0 0 0, axis 0 0 1, limit lower=0 upper=1
- added joint left_joint_4: type prismatic, parent left_forearm, child left_contact_4, origin xyz=-0.14999999999999997 0 -0.1 rpy=0 0 0, axis 0 0 0, limit lower=0 upper=1
- added joint right_joint_1: type prismatic, parent right_forearm, child right_contact_1, origin xyz=0.3 0 -0.1 rpy=0 0 0, axis 0 0 1, limit lower=0 upper=1
- added joint right_joint_2: type prismatic, parent right_forearm, child right_contact_2, origin xyz=0.25 0 -0.1 rpy=0 0 0, axis 0 0 1, limit lower=0 upper=1
- added joint right_joint_3: type prismatic, parent right_forearm, child right_contact_3, origin xyz=0.19999999999999998 0 -0.1 rpy=0 0 0, axis 0 0 1, limit lower=0 upper=1
- added joint right_joint_4: type prismatic, parent right_forearm, child right_contact_4, origin xyz=0.14999999999999997 0 -0.1 rpy=0 0 0, axis 0 0 1, limit lower=0 upper=1
- joint left_forearm_joint: axis 0 1 0 -> (none); type continuous -> fixed
- joint right_forearm_joint: axis 0 1 0 -> (none); type continuous -> fixed

File: temp_02.urdf (robot description, URDF)
Before this commit: robot test_obj, 1 links, 0 joints
Links:
- link obj_body: geometry collision sphere radius=0.2
